File: eagle/Mini-Mixer.brd (EAGLE design)
At the start: 54.3 x 26.7 mm, 14 parts, among them IC1 LM4558N

Commit message: Board Design Fix
Parts:
- removed U$1: TLE2426CLP, tle2426:TO226AA
- added C6, C7, C8: 10uF, rcl:TT2D4L
- added LED1: (no value), led:LED3MM
- added R4, R6: 22k, rcl:0207/7
- added R7: 10k, rcl:0207/7
- IC1: value LM4558N -> NJM2732
- moved C1 20.3 mm to (10.2, 25.4)
- moved R1 20.3 mm to (19.1, 25.4)
- moved JP4 10.2 mm to (44.5, 5.08), turned to 0 degrees
- moved C2 10.2 mm to (10.2, 20.3)
- moved R2 10.2 mm to (19.1, 20.3)
- moved JP1 7.62 mm to (2.54, 19.1), turned to 270 degrees
- moved C4 5.68 mm to (38.1, 16.5), turned to 270 degrees
- moved C5 5.68 mm to (25.4, 21.6), turned to 270 degrees
- moved IC1 5.68 mm to (31.8, 19.1)
- moved JP2 5.68 mm to (40.6, 21.6)
- moved R5 5.68 mm to (36.8, 25.4)
Connections:
- new net N$11: IC1.5, R4.1, R6.2
- net +5V: now also C4.2, C7.+, C8.+, R4.2, R7.2; no longer C4.1, U$1.3
- net AGND: now also C4.1, C6.+, C7.-, IC1.6, IC1.7; no longer C4.2, U$1.1
- net GND: now also C6.-, C8.-, LED1.K, R6.1; no longer IC1.6, U$1.2
- net N$8: now also LED1.A, R7.1; no longer IC1.5, IC1.7
Routing:
- net GND: track 0.00 -> 70.7 mm
- net AGND: track 0.00 -> 64.6 mm
- net +5V: track 0.00 -> 35.6 mm
- net N$7: track 10.2 -> 22.9 mm
- net N$11: track 0.00 -> 10.2 mm
- net N$9: track 0.00 -> 7.62 mm
- net N$8: track 0.00 -> 2.54 mm
- net N$1: track 7.62 -> 6.13 mm
- net N$3: track 7.62 -> 6.13 mm
Other:
- board size 54.3 x 26.7 mm -> 47.9 x 29.2 mm
