File: eagle/Mini-Mixer.sch (EAGLE design)
At the start: 14 parts, among them IC1 LM4558N

Commit message: Board Design Fix
Parts:
- removed U$1: TLE2426CLP, tle2426:TLE2426CLP
- added C6, C7, C8: 10uF, rcl:CPOL-EUTT2D4L
- added LED1: (no value), led:LED3MM
- added R4, R6: 22k, rcl:R-EU_0207/7
- added R7: 10k, rcl:R-EU_0207/7
- IC1: value LM4558N -> NJM2732
Connections:
- new net N$11: IC1B.+IN, R4.1, R6.2
- net +5V: now also C4.2, C7.+, C8.+, R4.2, R7.2; no longer C4.1, U$1.IN
- net AGND: now also C4.1, C6.+, C7.-, IC1B.-IN, IC1B.OUT; no longer C4.2, U$1.OUT
- net GND: now also C6.-, C8.-, LED1.C, R6.1; no longer IC1B.-IN, U$1.COM
- net N$8: now also LED1.A, R7.1; no longer IC1B.+IN, IC1B.OUT
Other:
- moved on the sheet: C4, C5, IC1B, JP4
